File: eagle/unified-board/baxandall.brd (EAGLE design)
At the start: 76.2 x 50.8 mm, 75 parts, among them IC101 THAT151x, J103 phantom, J104 eqout, J601 micout, U101 OPAMPLME49710, U601 LM3915N, U602 LM3915N, U603 OPAMPLME49710

Commit message: A couple more bits done up.
Parts:
- removed D601: RED, SparkFun-LED:LED_BARGRAPH_10
- removed U601: LM3915N, SparkFun-IC-Special-Function:DIL18
- added C3: 100pf, SparkFun-Capacitors:CAP-PTH-SMALL
- added D1: RECTIFIERRB15X, mixer:SM-RECTIFIER
- added FB1: FB, mixer:BEAD
- added R1, R2: ???, SparkFun-Resistors:AXIAL-0.3
- J601: value micout -> out2
Connections:
- removed net N$18: C602.2, J601.1
- removed net V+: U601.3, U602.3
- removed net V-: U601.2, U602.2
- new net N$11: C602.2, D1.AC1, D1.AC2, FB1.P$1, U602.5
- new net N$20: D602.11, U602.1
- new net N$41: D602.12, U602.18
- new net N$43: D602.13, U602.17
- new net N$44: D602.14, U602.16
- new net N$45: D602.15, U602.15
- new net N$46: D602.16, U602.14
- new net N$47: D602.17, U602.13
- new net N$48: D602.18, U602.12
- new net N$49: D602.19, U602.11
- new net N$50: D602.20, U602.10
- new net N$51: R1.P$1, U602.6, U602.7
- new net N$52: R1.P$2, R2.P$1, U602.8
- new net N$7: C3.1, FB1.P$2, J601.1
- net GND: now also C3.2, R2.P$2, U602.2
- net VCC: now also D1.POS, D602.1, D602.10, D602.2, D602.3, D602.4, D602.5, D602.6, D602.7, D602.8, D602.9, U602.3
- net VNEG: now also D1.NEG
