File: eagle/unified-board/unified.sch (EAGLE design)
At the start: 299 parts, among them IC101 THAT151x, IC201 THAT151x, IC301 THAT151x, IC401 THAT151x, J103 phantom, J104 eqout, J105 eqout, J203 phantom, J204 eqout, J205 eqout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

Commit message: Possibly complete?
doublechecked all IC footprints.
Routed the peak detector & found 1uf caps for it.
Parts:
- added C3, C4, C5, C6: 1uf/160V, mixer:CAP-LYTIC1UF/160V
Connections:
- new net N$38: C3.-, R4.1
- new net N$39: C4.+, R6.2, U502.SIGIN
- new net N$54: C5.-, R1.1
- net GND: now also C4.-, C6.-
- net N$11: now also C5.+; no longer R1.1
- net N$152: now also C3.+; no longer U502.SIGIN
- net N$23: now also C6.+
Other:
- moved on the sheet: D3, D4, D502, R4, R5, R509, R510, R511, R6, U1G2, U502

Commit message: More touchups.
Doublechecked rotary switch direction and values.
Added some dimension lines.
Parts:
- IC101, IC201, IC301, IC401: value THAT151x -> THAT1512; device mosfet:THAT151X -> mixer:THAT151X
Changed lines of the file:
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@@
 <part name="C115" library="mixer" deviceset="WIMA-MKS2" device="0.1UF" value="0.1uf"/>
 <part name="C116" library="mixer" deviceset="WIMA-MKS2" device="0.1UF" value="0.1uf"/>
-<part name="IC101" library="mosfet" deviceset="THAT151X" device="" value="THAT151x"/>
+<part name="IC101" library="mixer" deviceset="THAT151X" device="" value="THAT1512"/>
 <part name="D103" library="SparkFun-DiscreteSemi" deviceset="DIODE" device="-1N4148" value="200mA/100V/1V"/>
 <part name="D102" library="SparkFun-DiscreteSemi" deviceset="DIODE" device="-1N4148" value="200mA/100V/1V"/>
@@
 <part name="C215" library="mixer" deviceset="WIMA-MKS2" device="0.1UF" value="0.1uf"/>
 <part name="C216" library="mixer" deviceset="WIMA-MKS2" device="0.1UF" value="0.1uf"/>
-<part name="IC201" library="mosfet" deviceset="THAT151X" device="" value="THAT151x"/>
+<part name="IC201" library="mixer" deviceset="THAT151X" device="" value="THAT1512"/>
 <part name="D203" library="SparkFun-DiscreteSemi" deviceset="DIODE" device="-1N4148" value="200mA/100V/1V"/>
 <part name="D202" library="SparkFun-DiscreteSemi" deviceset="DIODE" device="-1N4148" value="200mA/100V/1V"/>
@@
 <part name="C315" library="mixer" deviceset="WIMA-MKS2" device="0.1UF" value="0.1uf"/>
 <part name="C316" library="mixer" deviceset="WIMA-MKS2" device="0.1UF" value="0.1uf"/>
-<part name="IC301" library="mosfet" deviceset="THAT151X" device="" value="THAT151x"/>
+<part name="IC301" library="mixer" deviceset="THAT151X" device="" value="THAT1512"/>
 <part name="D303" library="SparkFun-DiscreteSemi" deviceset="DIODE" device="-1N4148" value="200mA/100V/1V"/>
 <part name="D302" library="SparkFun-DiscreteSemi" deviceset="DIODE" device="-1N4148" value="200mA/100V/1V"/>
@@
 <part name="C415" library="mixer" deviceset="WIMA-MKS2" device="0.1UF" value="0.1uf"/>
 <part name="C416" library="mixer" deviceset="WIMA-MKS2" device="0.1UF" value="0.1uf"/>
-<part name="IC401" library="mosfet" deviceset="THAT151X" device="" value="THAT151x"/>
+<part name="IC401" library="mixer" deviceset="THAT151X" device="" value="THAT1512"/>
 <part name="D403" library="SparkFun-DiscreteSemi" deviceset="DIODE" device="-1N4148" value="200mA/100V/1V"/>
 <part name="D402" library="SparkFun-DiscreteSemi" deviceset="DIODE" device="-1N4148" value="200mA/100V/1V"/>

Commit message: Some updates.
-More BOM detail
-SVG for temp panel.
-Few more dimensions on board.
-Tweaking preamp gains on rotpot boards.
Parts:
- R701, R702: value 10r -> 10
Changed lines of the file:
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@@
 <part name="SUPPLY701" library="SparkFun-Aesthetics" deviceset="VCC" device=""/>
 <part name="J701" library="SparkFun-Connectors" deviceset="CONN_03" device="POLAR_LOCK" value="power"/>
-<part name="R701" library="SparkFun-Resistors" deviceset="RESISTOR" device="AXIAL-0.3" value="10r"/>
-<part name="R702" library="SparkFun-Resistors" deviceset="RESISTOR" device="AXIAL-0.3" value="10r"/>
+<part name="R701" library="SparkFun-Resistors" deviceset="RESISTOR" device="AXIAL-0.3" value="10"/>
+<part name="R702" library="SparkFun-Resistors" deviceset="RESISTOR" device="AXIAL-0.3" value="10"/>
 <part name="GND702" library="SparkFun-Aesthetics" deviceset="GND" device=""/>
 <part name="R703" library="SparkFun-Resistors" deviceset="RESISTOR" device="AXIAL-0.3" value="1k5"/>

Commit message: Many changes from checkplots.
Some footprints were incorrect.  Library, board & schem all updated.
Parts:
- removed H606, H607, H608, H609, H610: STAND-OFF, SparkFun-Hardware:STAND-OFF
Changed lines of the file:
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@@
 <part name="H612" library="SparkFun-Hardware" deviceset="STAND-OFF" device=""/>
 <part name="H611" library="SparkFun-Hardware" deviceset="STAND-OFF" device=""/>
-<part name="H609" library="SparkFun-Hardware" deviceset="STAND-OFF" device=""/>
-<part name="H610" library="SparkFun-Hardware" deviceset="STAND-OFF" device=""/>
-<part name="H608" library="SparkFun-Hardware" deviceset="STAND-OFF" device=""/>
-<part name="H607" library="SparkFun-Hardware" deviceset="STAND-OFF" device=""/>
 <part name="H605" library="SparkFun-Hardware" deviceset="STAND-OFF" device=""/>
-<part name="H606" library="SparkFun-Hardware" deviceset="STAND-OFF" device=""/>
 <part name="H604" library="SparkFun-Hardware" deviceset="STAND-OFF" device=""/>
 <part name="H603" library="SparkFun-Hardware" deviceset="STAND-OFF" device=""/>
@@
 <instance part="H612" gate="G$1" x="429.26" y="38.1"/>
 <instance part="H611" gate="G$1" x="429.26" y="40.64"/>
-<instance part="H609" gate="G$1" x="426.72" y="40.64"/>
-<instance part="H610" gate="G$1" x="426.72" y="38.1"/>
-<instance part="H608" gate="G$1" x="424.18" y="38.1"/>
-<instance part="H607" gate="G$1" x="424.18" y="40.64"/>
 <instance part="H605" gate="G$1" x="421.64" y="40.64"/>
-<instance part="H606" gate="G$1" x="421.64" y="38.1"/>
 <instance part="H604" gate="G$1" x="419.1" y="38.1"/>
 <instance part="H603" gate="G$1" x="419.1" y="40.64"/>

Commit message: Peppered the board with ground stitch vias.
Parts:
- removed H604, H611: STAND-OFF, SparkFun-Hardware:STAND-OFF
Changed lines of the file:
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@@
 <part name="R611" library="mixer" deviceset="RESISTOR" device="" value="???"/>
 <part name="H612" library="SparkFun-Hardware" deviceset="STAND-OFF" device=""/>
-<part name="H611" library="SparkFun-Hardware" deviceset="STAND-OFF" device=""/>
 <part name="H605" library="SparkFun-Hardware" deviceset="STAND-OFF" device=""/>
-<part name="H604" library="SparkFun-Hardware" deviceset="STAND-OFF" device=""/>
 <part name="H603" library="SparkFun-Hardware" deviceset="STAND-OFF" device=""/>
 <part name="H601" library="SparkFun-Hardware" deviceset="STAND-OFF" device=""/>
@@
 <instance part="R611" gate="G$1" x="325.12" y="185.42" rot="R180"/>
 <instance part="H612" gate="G$1" x="429.26" y="38.1"/>
-<instance part="H611" gate="G$1" x="429.26" y="40.64"/>
 <instance part="H605" gate="G$1" x="421.64" y="40.64"/>
-<instance part="H604" gate="G$1" x="419.1" y="38.1"/>
 <instance part="H603" gate="G$1" x="419.1" y="40.64"/>
 <instance part="H601" gate="G$1" x="416.56" y="40.64"/>

Commit message: Board touchups before gerbers.
Parts:
- removed VR104, VR105, VR204, VR205, VR304, VR305, VR404, VR405: 10K, mixer:POT10K-VERTPIN
Connections:
- net GND: no longer VR104.A, VR105.A, VR204.A, VR205.A, VR304.A, VR305.A, VR404.A, VR405.A
Changed lines of the file:
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@@
 <part name="D101" library="mixer" deviceset="RECTIFIER" device="RB15X"/>
 <part name="FRAME101" library="SparkFun-Aesthetics" deviceset="FRAME-LEDGER" device=""/>
-<part name="VR104" library="mixer" deviceset="POT" device="10K-VERTPIN" value="10K"/>
-<part name="VR105" library="mixer" deviceset="POT" device="10K-VERTPIN" value="10K"/>
 <part name="FRAME601" library="SparkFun-Aesthetics" deviceset="FRAME-LEDGER" device=""/>
 <part name="C602" library="mixer" deviceset="CAP-LYTIC" device="47U/25V" value="47u/25V"/>
@@
 <part name="GND107" library="SparkFun-Aesthetics" deviceset="GND" device=""/>
 <part name="GND606" library="SparkFun-Aesthetics" deviceset="GND" device=""/>
-<part name="GND106" library="SparkFun-Aesthetics" deviceset="GND" device=""/>
-<part name="GND108" library="SparkFun-Aesthetics" deviceset="GND" device=""/>
 <part name="SUPPLY205" library="SparkFun-Aesthetics" deviceset="VCC" device=""/>
 <part name="VR203" library="mixer" deviceset="POT" device="10K-VERTPIN" value="10K"/>
@@
 <part name="C214" library="mixer" deviceset="CAP-LYTIC" device="47U/25V" value="47u/25V"/>
 <part name="D201" library="mixer" deviceset="RECTIFIER" device="RB15X"/>
-<part name="VR204" library="mixer" deviceset="POT" device="10K-VERTPIN" value="10K"/>
-<part name="VR205" library="mixer" deviceset="POT" device="10K-VERTPIN" value="10K"/>
 <part name="C220" library="mixer" deviceset="CAP-LYTIC" device="47U/25V" value="47u/25V"/>
 <part name="J204" library="SparkFun-Connectors" deviceset="M01" device="NOSILK-KIT" value="eqout"/>
 <part name="J206" library="SparkFun-Connectors" deviceset="CONN_05" device="PTH_LONGPADS"/>
 <part name="GND207" library="SparkFun-Aesthetics" deviceset="GND" device=""/>
-<part name="GND206" library="SparkFun-Aesthetics" deviceset="GND" device=""/>
-<part name="GND208" library="SparkFun-Aesthetics" deviceset="GND" device=""/>
 <part name="SUPPLY305" library="SparkFun-Aesthetics" deviceset="VCC" device=""/>
 <part name="VR303" library="mixer" deviceset="POT" device="10K-VERTPIN" value="10K"/>
@@
 <part name="C314" library="mixer" deviceset="CAP-LYTIC" device="47U/25V" value="47u/25V"/>
 <part name="D301" library="mixer" deviceset="RECTIFIER" device="RB15X"/>
-<part name="VR304" library="mixer" deviceset="POT" device="10K-VERTPIN" value="10K"/>
-<part name="VR305" library="mixer" deviceset="POT" device="10K-VERTPIN" value="10K"/>
 <part name="C320" library="mixer" deviceset="CAP-LYTIC" device="47U/25V" value="47u/25V"/>
 <part name="J304" library="SparkFun-Connectors" deviceset="M01" device="NOSILK-KIT" value="eqout"/>
 <part name="J306" library="SparkFun-Connectors" deviceset="CONN_05" device="PTH_LONGPADS"/>
 <part name="GND307" library="SparkFun-Aesthetics" deviceset="GND" device=""/>
-<part name="GND306" library="SparkFun-Aesthetics" deviceset="GND" device=""/>
-<part name="GND308" library="SparkFun-Aesthetics" deviceset="GND" device=""/>
 <part name="SUPPLY405" library="SparkFun-Aesthetics" deviceset="VCC" device=""/>
 <part name="VR403" library="mixer" deviceset="POT" device="10K-VERTPIN" value="10K"/>
@@
 <part name="C414" library="mixer" deviceset="CAP-LYTIC" device="47U/25V" value="47u/25V"/>
 <part name="D401" library="mixer" deviceset="RECTIFIER" device="RB15X"/>
-<part name="VR404" library="mixer" deviceset="POT" device="10K-VERTPIN" value="10K"/>
-<part name="VR405" library="mixer" deviceset="POT" device="10K-VERTPIN" value="10K"/>
 <part name="C420" library="mixer" deviceset="CAP-LYTIC" device="47U/25V" value="47u/25V"/>
 <part name="J404" library="SparkFun-Connectors" deviceset="M01" device="NOSILK-KIT" value="eqout"/>
 <part name="J406" library="SparkFun-Connectors" deviceset="CONN_05" device="PTH_LONGPADS"/>
 <part name="GND407" library="SparkFun-Aesthetics" deviceset="GND" device=""/>
-<part name="GND406" library="SparkFun-Aesthetics" deviceset="GND" device=""/>
-<part name="GND408" library="SparkFun-Aesthetics" deviceset="GND" device=""/>
 <part name="C502" library="mixer" deviceset="CAP-LYTIC" device="47U/25V" value="47u/25V"/>
 <part name="GND501" library="SparkFun-Aesthetics" deviceset="GND" device=""/>
@@
 <instance part="FRAME101" gate="G$1" x="0" y="0"/>
 <instance part="FRAME101" gate="G$2" x="330.2" y="0"/>
-<instance part="VR104" gate="G$1" x="355.6" y="114.3"/>
-<instance part="VR105" gate="G$1" x="388.62" y="114.3"/>
 <instance part="C120" gate="G$1" x="340.36" y="175.26" rot="R90"/>
 <instance part="J104" gate="G$1" x="236.22" y="205.74" rot="R180"/>
 <instance part="J106" gate="G$1" x="373.38" y="152.4" rot="R180"/>
 <instance part="GND107" gate="1" x="363.22" y="142.24"/>
-<instance part="GND106" gate="1" x="355.6" y="104.14"/>
-<instance part="GND108" gate="1" x="388.62" y="104.14"/>
 </instances>
 <busses>
@@
 <wire x1="365.76" y1="147.32" x2="363.22" y2="147.32" width="0.1524" layer="91"/>
 <junction x="363.22" y="147.32"/>
-</segment>
-<segment>
-<pinref part="VR104" gate="G$1" pin="A"/>
-<pinref part="GND106" gate="1" pin="GND"/>
-</segment>
-<segment>
-<pinref part="VR105" gate="G$1" pin="A"/>
-<pinref part="GND108" gate="1" pin="GND"/>
 </segment>
 </net>
@@
 <instance part="C214" gate="G$1" x="210.82" y="208.28" rot="R90"/>
 <instance part="D201" gate="G$1" x="116.84" y="241.3" rot="MR90"/>
-<instance part="VR204" gate="G$1" x="353.06" y="116.84"/>
-<instance part="VR205" gate="G$1" x="386.08" y="116.84"/>
 <instance part="C220" gate="G$1" x="337.82" y="177.8" rot="R90"/>
 <instance part="J204" gate="G$1" x="233.68" y="208.28" rot="R180"/>
 <instance part="J206" gate="G$1" x="370.84" y="154.94" rot="R180"/>
 <instance part="GND207" gate="1" x="360.68" y="144.78"/>
-<instance part="GND206" gate="1" x="353.06" y="106.68"/>
-<instance part="GND208" gate="1" x="386.08" y="106.68"/>
 </instances>
 <busses>
@@
 <wire x1="363.22" y1="149.86" x2="360.68" y2="149.86" width="0.1524" layer="91"/>
 <junction x="360.68" y="149.86"/>
-</segment>
-<segment>
-<pinref part="VR204" gate="G$1" pin="A"/>
-<pinref part="GND206" gate="1" pin="GND"/>
-</segment>
-<segment>
-<pinref part="VR205" gate="G$1" pin="A"/>
-<pinref part="GND208" gate="1" pin="GND"/>
 </segment>
 </net>
@@
 <instance part="C314" gate="G$1" x="210.82" y="203.2" rot="R90"/>
 <instance part="D301" gate="G$1" x="116.84" y="236.22" rot="MR90"/>
-<instance part="VR304" gate="G$1" x="353.06" y="111.76"/>
-<instance part="VR305" gate="G$1" x="386.08" y="111.76"/>
 <instance part="C320" gate="G$1" x="337.82" y="172.72" rot="R90"/>
 <instance part="J304" gate="G$1" x="233.68" y="203.2" rot="R180"/>
 <instance part="J306" gate="G$1" x="370.84" y="149.86" rot="R180"/>
 <instance part="GND307" gate="1" x="360.68" y="139.7"/>
-<instance part="GND306" gate="1" x="353.06" y="101.6"/>
-<instance part="GND308" gate="1" x="386.08" y="101.6"/>
 </instances>
 <busses>
@@
 <wire x1="363.22" y1="144.78" x2="360.68" y2="144.78" width="0.1524" layer="91"/>
 <junction x="360.68" y="144.78"/>
-</segment>
-<segment>
-<pinref part="VR304" gate="G$1" pin="A"/>
-<pinref part="GND306" gate="1" pin="GND"/>
-</segment>
-<segment>
-<pinref part="VR305" gate="G$1" pin="A"/>
-<pinref part="GND308" gate="1" pin="GND"/>
 </segment>
 </net>
@@
 <instance part="C414" gate="G$1" x="210.82" y="200.66" rot="R90"/>
 <instance part="D401" gate="G$1" x="116.84" y="233.68" rot="MR90"/>
-<instance part="VR404" gate="G$1" x="353.06" y="109.22"/>
-<instance part="VR405" gate="G$1" x="386.08" y="109.22"/>
 <instance part="C420" gate="G$1" x="337.82" y="170.18" rot="R90"/>
 <instance part="J404" gate="G$1" x="233.68" y="200.66" rot="R180"/>
 <instance part="J406" gate="G$1" x="370.84" y="147.32" rot="R180"/>
 <instance part="GND407" gate="1" x="360.68" y="137.16"/>
-<instance part="GND406" gate="1" x="353.06" y="99.06"/>
-<instance part="GND408" gate="1" x="386.08" y="99.06"/>
 </instances>
 <busses>
@@
 <junction x="360.68" y="142.24"/>
 </segment>
-<segment>
-<pinref part="VR404" gate="G$1" pin="A"/>
-<pinref part="GND406" gate="1" pin="GND"/>
-</segment>
-<segment>
-<pinref part="VR405" gate="G$1" pin="A"/>
-<pinref part="GND408" gate="1" pin="GND"/>
-</segment>
-</net>
+</net>
